Commit message: update

File: isaac_sim_test_description/urdf/isaac_sim_test.urdf (robot description, URDF)
Before this commit: robot isaac_sim_test, 2 links, 1 joints
Joints:
- removed joint ��] 1
- added joint joint_1: type continuous, parent base_link, child hoge_link_1, origin xyz=0.0 0.0 0.0 rpy=0 0 0, axis 0.0 0.0 1.0

File: isaac_sim_test_description/urdf/materials.xacro (robot description, xacro)
@@ -1,6 +1,6 @@
 <?xml version="1.0" ?>
-<robot name="isaac_sim_test" xmlns:xacro="http://www.ros.org/wiki/xacro" >
-<material name="silver">
-  <color rgba="0.700 0.700 0.700 1.000"/>
-</material>
+<robot xmlns:xacro="http://www.ros.org/wiki/xacro">
+  <material name="silver">
+    <color rgba="0.75 0.75 0.75 1.0"/>
+  </material>
 </robot>
